File: battery replacement.kicad_sch (KiCad schematic)
At the start: 15 parts, among them U1 GP3134_C48997205

Commit message: prelim. 10x25mm ~ 180pcs
Parts:
- removed L1: 4.7uH, JLCImport:BMQA000606304R7MA1, symbol JLCImport:BMQA000606304R7MA1
- removed R1, R4: 10k, JLCImport:0402WGF1002TCE, symbol JLCImport:0402WGF1002TCE
- removed R2, R3: 20k, JLCImport:0402WGF2002TCE, symbol JLCImport:0402WGF2002TCE
- removed U1: GP3134_C48997205, JLCImport:GP3134_C48997205, symbol JLCImport:GP3134_C48997205
- added C7: 4.7uF, JLCImport:CL21A475KAQNNNE, symbol JLCImport:CL21A475KAQNNNE
- added L1: 470nH, JLCImport:TMS252012ALM-R47MTAA, symbol JLCImport:TMS252012ALM-R47MTAA
- added R1, R3: 100k, JLCImport:0402WGF1003TCE, symbol JLCImport:0402WGF1003TCE
- added R2: 549k, JLCImport:0402WGF5493TCE, symbol JLCImport:0402WGF5493TCE
- added U1: RT5788BGJ8F, JLCImport:RT5788BGJ8F, symbol JLCImport:RT5788BGJ8F
- added U2: Y4203-ADJM6R, JLCImport:Y4203-ADJM6R, symbol JLCImport:Y4203-ADJM6R
Connections:
- net BS is gone; now on net GND: C2.2
- net SW is gone; now on net +5V: C2.1
- net +5V: now also C1.2, R3.2, U1.2 (VIN), U2.3 (OUT); no longer C1.1, USB1.A9 (VBUS), USB1.B9 (VBUS)
- net EN: now also R3.1, U1.8 (EN)
- net FB: now also R1.1, R2.1, U1.7 (FB)
- net GND: now also C1.1, C7.1, U2.1 (OVLO), U2.6 (GND); no longer C1.2
- net V_OUT renamed VOUT
- net VOUT: now also L1.2, R2.2, U1.5 (VOUT)
- new net AGND: R1.2, U1.6 (AGND)
- new net LX: L1.1, U1.3 (LX)
- new net PGND: U1.4 (PGND)
- new net VBUS: C7.2, U2.4 (VIN), U2.5 (VCC), USB1.A9 (VBUS), USB1.B9 (VBUS)
- no-connect marks 0 -> 2
Other:
- note added: "TODO: light up a LED when PGOOD"
- note added: "The converter needs 22uF + 100nF on it's input. USB permits only 10uF, so this load switch charges the input caps slowly."
- note removed: "TestPoints are only for soldering cables"
- moved on the sheet: C1, C2, C3, C4, R5, R6, TP1, TP2, USB1

Commit message: prelim 9x25mm ~ 200pcs
Connections:
- net AGND is gone; now on net GND: R1.2, U1.6 (AGND)
- net PGND is gone; now on net GND: U1.4 (PGND)
Changed lines of the file:
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@@
+	)
+	(junction
+		(at 248.92 82.55)
+		(diameter 0)
+		(color 0 0 0 0)
 	)
 	(junction
@@
 	(wire
 		(pts
+			(xy 248.92 82.55) (xy 248.92 83.82)
+		)
+		(stroke
+			(width 0)
+			(type default)
+		)
+	)
+	(wire
+		(pts
 			(xy 34.29 45.72) (xy 34.29 35.56)
 		)
@@
 		(pts
 			(xy 237.49 36.83) (xy 243.84 36.83)
+		)
+		(stroke
+			(width 0)
+			(type default)
+		)
+	)
+	(wire
+		(pts
+			(xy 274.32 82.55) (xy 280.67 82.55)
 		)
 		(stroke
@@
 			)
 			(justify left bottom)
+		)
+	)
+	(label "PGND"
+		(at 280.67 82.55 180)
+		(effects
+			(font
+				(size 1.27 1.27)
+			)
+			(justify right bottom)
 		)
 	)
@@
 					(unit 1)
 				)
+			)
+		)
+	)
+	(symbol
+		(lib_id "power:GND")
+		(at 248.92 83.82 0)
+		(unit 1)
+		(body_style 1)
+		(exclude_from_sim no)
+		(in_bom yes)
+		(on_board yes)
+		(in_pos_files yes)
+		(dnp no)
+		(fields_autoplaced yes)
+		(property "Reference" "#PWR04"
+			(at 248.92 90.17 0)
+			(hide yes)
+			(show_name no)
+			(do_not_autoplace no)
+			(effects
+				(font
+					(size 1.27 1.27)
+				)
+			)
+		)
+		(property "Value" "GND"
+			(at 248.92 88.9 0)
+			(show_name no)
+			(do_not_autoplace no)
+			(effects
+				(font
+					(size 1.27 1.27)
+				)
+			)
+		)
+		(property "Footprint" ""
+			(at 248.92 83.82 0)
+			(hide yes)
+			(show_name no)
+			(do_not_autoplace no)
+			(effects
+				(font
+					(size 1.27 1.27)
+				)
+			)
+		)
+		(property "Datasheet" ""
+			(at 248.92 83.82 0)
+			(hide yes)
+			(show_name no)
+			(do_not_autoplace no)
+			(effects
+				(font
+					(size 1.27 1.27)
+				)
+			)
+		)
+		(property "Description" "Power symbol creates a global label with name \"GND\" , ground"
+			(at 248.92 83.82 0)
+			(hide yes)
+			(show_name no)
+			(do_not_autoplace no)
+			(effects
+				(font
+					(size 1.27 1.27)
+				)
+			)
+		)
+		(pin "1"
+		)
+		(instances
+			(project "battery replacement"
+				(path "/e18ffe70-5d49-4f98-b8fd-2f3dffb253f2"
+					(reference "#PWR04")
+					(unit 1)
+				)

Commit message: kicad prelim version
Parts:
- renumbered C7 to C1, C1 to C2, C2 to C3, C3 to C4, C4 to C5, R5 to R1, R6 to R2, R2 to R4, R1 to R5, U2 to U1, U1 to U2
Other:
- note added: "TODO: light up an LED when PGOOD"
- note removed: "TODO: light up a LED when PGOOD"
- title: (none) -> Battery replacement
- moved on the sheet: C2, C3, C4, C5, L1, R3, R4, R5, TP1, TP2, U2
